File: MSXMouseCH32V103C.kicad_sch (KiCad schematic)
At the start: 43 parts, among them J1 SW, J2 USART1, J3 DE9_Plug, J4 USB_1, J5 Conn_01x03, SW1 SW_Push, SW2 BOOT0, U1 CH32V203C8T6-CH32V103C, U2 LM1117MP-3.3, Y1 Crystal

Commit message: Project Rename
Parts:
- removed J1: SW, Connector_PinHeader_2.54mm:PinHeader_1x02_P2.54mm_Vertical, symbol Connector_Generic:Conn_01x02
- removed J2: USART1, Connector_PinHeader_2.54mm:PinHeader_1x02_P2.54mm_Vertical, symbol Connector_Generic:Conn_01x02
- removed JP2: Jumper_2_Open, Jumper:SolderJumper-2_P1.3mm_Open_RoundedPad1.0x1.5mm, symbol Jumper:Jumper_2_Open
- removed R3: R, Resistor_SMD:R_0805_2012Metric_Pad1.20x1.40mm_HandSolder, symbol Device:R
- added J1: Conn_01x04, Connector_PinHeader_2.54mm:PinHeader_1x04_P2.54mm_Vertical, symbol Connector_Generic:Conn_01x04
Connections:
- net CONF1: now also U1.22 (PB11); no longer U1.28 (PB15)
- net LED1: now also U1.46 (PB9); no longer U1.26 (PB13)
- net LED3: now also U1.3 (PC14_OSC32IN); no longer U1.27 (PB14)
- net PA10: now also J1.3 (Pin_3)
- net PA9: now also J1.4 (Pin_4)
- net SWCLK: now also J1.1 (Pin_1)
- net SWDIO: now also J1.2 (Pin_2)
- net CONF2: no longer names the net of U1.29 (PA8)
- no-connect marks 16 -> 17
